File: Hardware/Amplifierv0.2/Amplifierv0.2.kicad_sch (KiCad schematic)
At the start: 28 parts, among them J1 AudioJack2_Ground, J2 AudioJack3_Ground, Q1 NMOS, Q2 NMOS, U1 LM555xM, U2 LM78L05_SO8, U3 NJM4558, U4 74HCT04, U5 74LS04, U6 HIP2101_SOIC

Commit message: update schematic ampli
Parts:
- removed C2: 1nF, symbol Device:C
- removed J1: AudioJack2_Ground, symbol Connector_Audio:AudioJack2_Ground
- removed J2: AudioJack3_Ground, symbol Connector_Audio:AudioJack3_Ground
- removed L1: 6R8, symbol Device:L
- removed R1, R2, R6: 10k, symbol Device:R
- removed R3: 2k, symbol Device:R
- removed R4, R5: 10 Ω, symbol Device:R
- removed U4: 74HCT04, symbol 74xx:74HCT04
- removed U5: 74LS04, symbol 74xx:74LS04
- added C2: 1nf, symbol Device:C_Small
- added C?: 1000u, symbol Device:C
- added L?: 6R8, symbol Device:L_Small
- added R3: 2k, symbol Device:R_Small
- added R4, R5: 10, symbol Device:R_Small
- added R6, R7: 10k, symbol Device:R_Small
- added U? (x2): NJM4558, symbol Amplifier_Operational:NJM4558
Connections:
- net V_speakers is gone; now on net V_batterie: Q1.1 (D)
- net 0: now also C2.1; no longer C1.2, C3.2, C5.2, LS1.2, LS2.2, Q2.3 (S), RV10k.3, U2.2 (GND), U2.3 (GND), U2.6 (GND), U2.7 (GND), U3.4 (V-), U6.7 (VSS)
- net 5V: now also U?.8 (V+)
- net at U1.3 (Q): now also R3.2
- net V_comparateur1: now reaches U1.2 (TR), U1.6 (THR), U3.2 (-)
- net V_comparateur1: now also C2.2, R3.1, U?.3 (+)
- net V_HO: now reaches D2.1 (K), U6.3 (HO)
- net V_HO: now also R5.1
- net at D2.2 (A), Q1.2 (G): now also R5.2
- net at U6.6 (LI): now also U?.1
- net at LS1.1, LS2.1: now also C?.2; no longer C5.1
- net V_HP: now reaches C4.2, C6.2, Q1.3 (S), Q2.1 (D), U6.4 (HS)
- net V_HP: now also L?.1
- net V_LO: now reaches D1.1 (K), U6.8 (LO)
- net V_LO: now also R4.1
- net V_comparateur2: now reaches RV10k.2, U3.3 (+)
- net V_comparateur2: now also R6.1, R7.1, U?.2 (-)
- net at D1.2 (A), Q2.2 (G): now also R4.2
- net VBat renamed V_batterie
- new net: C5.1, C?.1, L?.2
- new net GND: C1.2, C3.2, C5.2, LS1.2, LS2.2, Q2.3 (S), RV10k.3, U2.2 (GND), U2.3 (GND), U2.6 (GND), U2.7 (GND), U3.4 (V-), U6.7 (VSS), U?.4 (V-)
- new net V_x: R6.2, R7.2
- no-connect marks 0 -> 1
Other:
- note added: "Amplificateur de classe D"
- note added: "Régulateur"
- note added: "Sortie haut-parleur"
- note added: "générateur de triangles"
- note added: "mosfet driver"
- note added: "transistor NMOS"
- moved on the sheet: C1, C3, C4, C5, C6, D1, D2, LS1, LS2, Q1, Q2, RV10k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
