File: Hardware/Amplifierv0.2/Amplifierv0.2 (2).kicad_sch (KiCad schematic)
At the start: 31 parts, among them Q1 NMOS, Q2 NMOS, U1 LM555xM, U2 LM78L05_SO8, U3 NJM4558, U6 HIP2101_SOIC

Commit message: updated amplifier schematic v3
Parts:
- gave numbers to parts that had none: 2
Other:
- note added: "STM32"
- moved on the sheet: C1, C2, C3, C4, C5, C6, C7, D1, D2, H1, H2, H3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
