File: Hardware/Amplifierv0.2/Amplifierv0.2 (2) (1) (1).kicad_sch (KiCad schematic)
At the start: 68 parts, among them IC1 TCPP01-M12, J1 Conn_01x03, J2 Conn_01x03, J3 USB_C_Receptacle, Q1 SI2304DDS-T1-GE3, Q2 SI2304DDS-T1-GE3, U1 SI2303CDS-T1-GE3, U3 SI2303CDS-T1-GE3, U4 STM32G491CETx (x=6), U6 SGTL5000XNLA3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

Commit message: apli v7
Parts:
- removed Q1: SI2304DDS-T1-GE3, Package_TO_SOT_SMD:SOT-23, symbol SI2304DDS:SI2304DDS-T1-GE3
- removed U1, U3: SI2303CDS-T1-GE3, Package_TO_SOT_SMD:SOT-23, symbol SI2303CDS:SI2303CDS-T1-GE3
- added C19: 1.1u, Capacitor_SMD:C_0603_1608Metric_Pad1.08x0.95mm_HandSolder, symbol Device:C_Small
- added C20, C23: 5u, Capacitor_SMD:C_0603_1608Metric_Pad1.08x0.95mm_HandSolder, symbol Device:C_Small
- added Q1, Q4: SI2303CDS-T1-GE3, symbol Simulation_SPICE:PMOS
- added Q3: SI2304DDS-T1-GE3, Package_TO_SOT_SMD:SOT-23, symbol Simulation_SPICE:NMOS
- C21: value 0.1 u -> 0.1u
- C22: value 1.0 u -> 1.0u
Connections:
- net 1.8V: now also U6.20 (VDDD)
- net 3.3VDC: now also U4.1 (VBAT), U4.20 (VREF+), U4.21 (VDDA), U4.24 (VDD), U4.36 (VDD), U4.48 (VDD), U6.12 (VDDIO), U6.3 (VDDA), C19.2, C20.1, C23.1
- net GND: now also U4.19 (VSSA), U4.23 (VSS), U4.35 (VSS), U4.47 (VSS), U6.21 (GND), C19.1, C20.2, C23.2, Q4.1 (D)
- net I2C_SGTL5000: no longer U4.44 (PB7)
- net SYS_MCLK: now also U6.13 (SYS_MCLK)
- net V_AMPLIFIER: now also Q3.3 (S), Q4.3 (S)
- net V_BAT+: now also Q1.1 (D)
- net V_SYS: now also Q1.3 (S), Q3.1 (D)
- net band1: now reaches U4.10 (PA2)
- net band3: now reaches U4.27 (PB13)
- net band2: now reaches U4.29 (PB15)
- net at R4.2: now also Q4.2 (G)
- net at D4.1 (K), R16.2: now also Q1.2 (G)
- net at R5.2: now also Q3.2 (G)
- no-connect marks 13 -> 20
Other:
- moved on the sheet: C21, C22
