File: Hardware/mainnboard_v1.4/Pojet 1A.kicad_pcb (KiCad board)
At the start: 4 copper layers, 60 x 60 mm, 92 parts, among them IC1 TCPP01-M12, J1 USB_C_Receptacle, J10 Conn_01x10, J2 Conn_ST_STDC14, J3 Conn_01x02, J4 Conn_01x02, J5 Conn_01x02, J7 Conn_01x05, J8 AudioJack3, J9 Conn_01x05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

Commit message: Add files via upload
update 1 error
Routing:
- net GND: track 43.1 -> 42.2 mm
