File: Hardware/SecondaryBoard/SecondaryBoard/SecondaryBoard.kicad_sch (KiCad schematic)
At the start: 21 parts, among them J1 Conn_01x10, J2 Conn_01x10

Commit message: update pff
Parts:
- removed J1, J2: Conn_01x10, symbol Connector_Generic:Conn_01x10
- added C5: 100nF, Capacitor_SMD:C_0603_1608Metric_Pad1.08x0.95mm_HandSolder, symbol Device:C
- added J4, J5: Conn_01x08, Connector_JST:JST_XH_B8B-XH-AM_1x08_P2.50mm_Vertical, symbol Connector_Generic:Conn_01x08
- added R10, R13, R14: 180, symbol Device:R
- added R11: 120, symbol Device:R
- added R12, R15, R16, R9: 160, symbol Device:R
- C1, C2, C3, C4: footprint (none) -> Capacitor_SMD:C_0603_1608Metric_Pad1.08x0.95mm_HandSolder
- D1: value LED -> Green
- D2: value LED -> Yellow
- D3: value LED -> Orange
- D4: value LED -> Red
- R1, R2, R3, R4, R5, R6, R7, R8: value 4.7k -> 10k; footprint (none) -> Resistor_SMD:R_0603_1608Metric_Pad0.98x0.95mm_HandSolder
- RV1: value R_Potentiometer -> B10K; footprint (none) -> WITNS:Potentiometer_Alpha_RD901F-40-00D_Single_Vertical
Connections:
- net +3.3V: now also J5.1 (Pin_1), R13.2, R14.2, R15.1, R16.2; no longer D1.2 (A), D2.2 (A), D3.2 (A), D4.2 (A)
- net A Encodeur 1: now also J4.1 (Pin_1)
- net A Encodeur 2: now also J4.4 (Pin_4)
- net B Encodeur 1: now also J4.2 (Pin_2)
- net B Encodeur 2: now also J4.3 (Pin_3)
- net EQ_BAND_BTN: now also J5.3 (Pin_3)
- net GND: now also C5.1, J5.8 (Pin_8)
- net Potar_volume: now also C5.2, J5.2 (Pin_2)
- net TIM3_CH1: now also J4.5 (Pin_5), R10.2; no longer S1.2
- net TIM3_CH2: now also J4.6 (Pin_6), R9.2; no longer S1.1
- net TIM3_CH3: now also J4.7 (Pin_7), R11.1; no longer S2.4
- net TIM3_CH4: now also J4.8 (Pin_8), R12.1; no longer S2.1
- net band0: now also J5.7 (Pin_7)
- net band1: now also J5.6 (Pin_6)
- net band2: now also J5.5 (Pin_5)
- net band3: now also J5.4 (Pin_4)
- new net: D2.2 (A), R14.1
- new net: R9.1, S1.1
- new net: R10.1, S1.2
- new net: R12.2, S2.1
- new net: R11.2, S2.4
- new net: D4.2 (A), R16.1
- new net: D1.2 (A), R13.1
- new net: D3.2 (A), R15.2
- no-connect marks 7 -> 3
Other:
- moved on the sheet: D1, D2, D3, D4

Commit message: Finished Update
Parts:
- added H1, H2, H3: MountingHole_Pad, MountingHole:MountingHole_3.2mm_M3_DIN965_Pad, symbol Mechanical:MountingHole_Pad
- D1: footprint LED_THT:LED_D5.0mm -> LED_THT:LED_D3.0mm
- D2, D3, D4: footprint (none) -> LED_THT:LED_D5.0mm
- R10, R11, R12, R13, R14, R15, R16, R9: footprint (none) -> Resistor_SMD:R_0603_1608Metric_Pad0.98x0.95mm_HandSolder
- S1, S2: footprint ENCODER_LED_3 -> WITNS:ENCODER_LED_3
Connections:
- net GND: now also H1.1, H2.1, H3.1
Other:
- note added: "Mounting holes"
