File: Hardware/SecondaryBoard/SecondaryBoard.kicad_pcb (KiCad board)
At the start: 2 copper layers, 85 x 31 mm, 33 parts, among them J4 Conn_01x08, J5 Conn_01x08

Commit message: last gerber vias and track size edits
Routing:
- net +3.3V: track 235.4 -> 236.2 mm
- net GND: vias 26 -> 28

Commit message: Final edit for building conformity
Routing:
- net +3.3V: track 236.2 -> 180.6 mm
- net Potar_volume: track 65.9 -> 62.2 mm
- net B Encodeur 1: track 42.5 -> 40.1 mm
- net EQ_BAND_BTN: vias 0 -> 1
- net A Encodeur 1: vias 0 -> 1
- net GND: vias 28 -> 36
